File: SD04Proto/boost.kicad_sch (KiCad schematic)
At the start: 33 parts, among them IC5 UCC28C50DGKR, Q1 2N7002BKVL, Q2 2N7002BKVL, Q3 BSC12DN20NS3GATMA1, Q4 2N7002BKVL, U2 SN74LVC1G125DCK

Commit message: updated layout after review
Parts:
- added C4: 470u, Capacitor_SMD:CP_Elec_10x10, symbol Device:C_Polarized
Connections:
- net 12V_Filt: now also C4.1
- net GND: now also C4.2

Commit message: Changed mosfet schematic symbol
Parts:
- Q3: footprint SamacSys_Parts:PG-TDSON-8_1 -> PG-TDSON-8_1
Connections:
- net 1Mhz_Switch_Sig: now reaches IC5.6 (OUT), Q3.4 (G)
- net 1Mhz_Switch_Sig: no longer Q3.2 (S), Q3.3 (S)
- net at D2.2 (A), L1.2, Q3.5 (D)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: now also Q3.9 (pad)
Changed lines of the file:
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@@
+		)
+	)
+	(label "1Mhz_Switch_Sig"
+		(at 107.95 121.92 0)
+		(effects
+			(font
+				(size 1.27 1.27)
+			)
+			(justify left bottom)
 		)
 	)
@@
 			)
 		)
-		(property "Footprint" "SamacSys_Parts:PG-TDSON-8_1"
+		(property "Footprint" "PG-TDSON-8_1"
 			(at 113.03 215.57 0)
 			(effects
@@
 		(pin "1"
 		)
-		(pin "2"
-		)
-		(pin "3"
+		(pin "9"
 		)
 		(pin "4"
